Commit message: v0.0.2

File: my_robot/urdf/my_robot.xacro (robot description, xacro)
@@ -22,5 +22,5 @@
       <origin xyz="0 0 0" rpy=" 0 0 0"/>
       <geometry>
-        <box size=".4 .2 .1"/>
+        <cylinder radius="0.2" length="0.1" />
       </geometry>
     </collision>
@@ -28,5 +28,5 @@
       <origin xyz="0 0 0" rpy=" 0 0 0"/>
       <geometry>
-        <box size=".4 .2 .1"/>
+        <cylinder radius="0.2" length="0.1" />
       </geometry>
     </visual>
@@ -57,5 +57,5 @@
   </link>
 <gazebo reference="chassis">
-    <material>Gazebo/Blue</material>
+    <material>Gazebo/Yellow</material>
 </gazebo>
 <link name='left_wheel'>
@@ -78,5 +78,5 @@
 </link>
 <gazebo reference="left_wheel">
-    <material>Gazebo/Green</material>
+    <material>Gazebo/Black</material>
 </gazebo>
 <link name='right_wheel'>
@@ -99,8 +99,8 @@
   </link>
 <gazebo reference="right_wheel">
-    <material>Gazebo/Green</material>
+    <material>Gazebo/Black</material>
 </gazebo>
  <joint type="continuous" name="left_wheel_hinge">
-    <origin xyz="0 0.15 0" rpy="0 0 0"/>
+    <origin xyz="0 0.25 0" rpy="0 0 0"/>
     <child link="left_wheel"/>
     <parent link="chassis"/>
@@ -110,5 +110,5 @@
   </joint>
  <joint type="continuous" name="right_wheel_hinge">
-    <origin xyz="0 -0.15 0" rpy="0 0 0"/>
+    <origin xyz="0 -0.25 0" rpy="0 0 0"/>
     <child link="right_wheel"/>
     <parent link="chassis"/>
@@ -136,5 +136,5 @@
   </link>
 <gazebo reference="camera">
-    <material>Gazebo/Red</material>
+    <material>Gazebo/Purple</material>
 </gazebo>
  <joint type="fixed" name="camera_joint">

Commit message: v0.0.2

File: my_robot/urdf/my_robot.xacro (robot description, xacro)
@@ -71,9 +71,15 @@
     </inertial>
     <visual name='left_wheel_visual'>
-      <origin xyz="0 0 0" rpy=" 0 1.5707 1.5707"/>
+      <origin xyz="0 0 0" rpy="0 1.5707 1.5707"/>
       <geometry>
           <cylinder radius="0.1" length="0.05" />
       </geometry>
     </visual>
+    <collision name='collision'>
+      <origin xyz="0 0 0" rpy="0 1.5707 1.5707"/>
+      <geometry>
+        <cylinder radius="0.1" length="0.05" />
+      </geometry>
+    </collision>
 </link>
 <gazebo reference="left_wheel">
@@ -92,9 +98,15 @@
     </inertial>
     <visual name='right_wheel_visual'>
-      <origin xyz="0 0 0" rpy=" 0 1.5707 1.5707"/>
+      <origin xyz="0 0 0" rpy="0 1.5707 1.5707"/>
       <geometry>
          <cylinder radius="0.1" length="0.05" />
       </geometry>
     </visual>
+    <collision name='collision'>
+      <origin xyz="0 0 0" rpy="0 1.5707 1.5707"/>
+      <geometry>
+        <cylinder radius="0.1" length="0.05" />
+      </geometry>
+    </collision>
   </link>
 <gazebo reference="right_wheel">
@@ -134,4 +146,10 @@
       </geometry>
     </visual>
+    <collision name='collision'>
+      <origin xyz="0 0 0" rpy=" 0 0 0"/>
+      <geometry>
+        <box size=".05 .05 .05"/>
+      </geometry>
+    </collision>
   </link>
 <gazebo reference="camera">
